File: file/pcb/v2/5x6/TPS/TPS.kicad_pcb (KiCad board)
At the start: 2 copper layers, 164 x 95.2 mm, 111 parts, among them J1 I2C, J10 AudioJack4, J2 FFC-0.5mm, 12p, J3 FFC-0.5mm, 12p, J4 PH2.0-2pin, J5 FFC-0.5mm, 6p, J6 FFC-0.5mm, 6p, J9 AudioJack4, K1 SW_Push, K10 SW_Push, K11 SW_Push, K12 SW_Push, K13 SW_Push, K14 SW_Push, K15 SW_Push, K16 SW_Push, K17 SW_Push, K18 SW_Push, K19 SW_Push, K2 SW_Push, K20 SW_Push, K21 SW_Push, K22 SW_Push, K23 SW_Push, K24 SW_Push, K25 EC-11, K26 SW_Push, K27 SW_Push, K28 SW_Push, K29 SW_Push, K3 SW_Push, K30 SW_Push, K31 SW_Push, K4 SW_Push, K5 SW_Push, K6 SW_Push, K7 SW_Push, K8 SW_Push, K9 SW_Push, SW1 SW_Push, SW2 MSKT-12D14, SW3 MSKT-12D14, U1 MCU_ProMicro_13p

Commit message: manufacturered with JLCPCB
Parts:
- removed H14, H15, H16 (x2), H17: edge, DreaM117er-keebLibrary:Breakaway_Tabs_2
- removed K20: SW_Push, DreaM117er-keebLibrary:SW_Hotswap_KLP12_GLP3.0_MX_Plated_1.00u_Dualside
- added HM1: MountingHole, ncParts:MountingHole_2.2mm_M2_ISO7380_Pad_noSilk, F.Cu at (107.2, 48.0)
- added HM2: MountingHole, ncParts:MountingHole_2.2mm_M2_ISO7380_Pad_noSilk, F.Cu at (111.9, 114.7)
- added HM3: MountingHole, ncParts:MountingHole_2.2mm_M2_ISO7380_Pad_noSilk, F.Cu at (164.3, 48.0)
- added HM5: MountingHole, ncParts:MountingHole_2.2mm_M2_ISO7380_Pad_noSilk, F.Cu at (183.4, 48.0)
- added HM6: MountingHole, ncParts:MountingHole_2.2mm_M2_ISO7380_Pad_noSilk, F.Cu at (178.6, 114.7)
- D1, D10, D11, D12, D13, D14, D15, D16, D17, D18, D19, D2, D20, D21, D22, D23, D24, D25, D26, D27, D28, D29, D3, D30, D31, D4, D5, D6, D7, D8, D9: footprint DreaM117er-keebLibrary:D_SOD-123_handsolder_dual -> ncParts-reversible:D3_TH_SMD_v2-reversible
- K1, K11, K12, K13, K14, K15, K16, K17, K18, K19, K2, K21, K22, K23, K24, K27, K28, K29, K3, K30, K4, K6, K7, K8, K9: footprint DreaM117er-keebLibrary:SW_Hotswap_KLP12_GLP3.0_MX_Plated_1.00u_Dualside -> ncSwitches:SW_hotswap_HLP_Plated_1u-reversible
- K10, K26, K31, K5: footprint DreaM117er-keebLibrary:SW_Hotswap_KLP12_GLP3.0_MX_Plated_1.00u_Dualside -> ncSwitches:SW_hotswap_HLP_Plated_1.25u-reversible
- moved D15 9.53 mm to (145.3, 106.2)
- moved K15 9.53 mm to (145.3, 114.7)
- moved D26 7.27 mm to (166.7, 106.2)
- moved D10 7.14 mm to (123.8, 106.2)
- moved K10 7.14 mm to (123.8, 114.7)
- moved K26 7.14 mm to (166.7, 114.7)
- moved D31 2.38 mm to (190.5, 106.2)
- moved D5 2.38 mm to (100.0, 106.2)
- moved K31 2.38 mm to (190.5, 114.7)
- moved K5 2.38 mm to (100.0, 114.7)
- moved D20 1.59 mm to (156.4, 106.2)
Connections:
- D20 pad 2: Net-(D20-Pad2) -> col2
- J4 pad 1: Net-(J4-Pin_1) -> BAT+
- J4 pad 2: BAT- -> GND
- J5 pad 1: SDA -> unconnected-(J5-Pin_1-Pad1)
- J5 pad 2: SCL -> unconnected-(J5-Pin_2-Pad2)
- J5 pad 3: +3V3 -> GND
- J5 pad 4: GND -> +3V3
- J5 pad 5: unconnected-(J5-Pin_5-Pad5) -> SCL
- J5 pad 6: unconnected-(J5-Pin_6-Pad6) -> SDA
- J5 pad 7: GND -> unconnected-(J5-Pin_7-Pad7)
- J6 pad 1: SDA -> unconnected-(J6-Pin_1-Pad1)
- J6 pad 2: SCL -> unconnected-(J6-Pin_2-Pad2)
- J6 pad 3: +3V3 -> GND
- J6 pad 4: GND -> +3V3
- J6 pad 5: unconnected-(J6-Pin_5-Pad5) -> SCL
- J6 pad 6: unconnected-(J6-Pin_6-Pad6) -> SDA
- J6 pad 7: GND -> unconnected-(J6-Pin_7-Pad7)
- J7 pad 1: Net-(J7-Pin_1) -> BAT+
- J7 pad 2: BAT- -> GND
- J8 pad 1: BAT- -> GND
- J8 pad 2: Net-(J7-Pin_1) -> BAT+
- SW2 pad 1: BAT+ -> RAW
- SW2 pad 2: Net-(J4-Pin_1) -> BAT+
- SW3 pad 1: BAT+ -> RAW
- SW3 pad 2: Net-(J7-Pin_1) -> BAT+
- U1 pad 1: BAT- -> unconnected-(U1-?-Pad1)
- U1 pad 26: BAT+ -> unconnected-(U1-?-Pad26)
Routing:
- net RAW: track 49.4 -> 214.8 mm, vias 2 -> 4
- net BAT-: track 149.9 -> 0.00 mm, vias 2 -> 0
- net GND: track 45.9 -> 131.0 mm, vias 21 -> 45
- net Net-(J4-Pin_1): track 65.9 -> 0.00 mm, vias 1 -> 0
- net BAT+: track 179.4 -> 131.4 mm, vias 4 -> 2
- net SCL: track 174.6 -> 135.4 mm, vias 3 -> 4
- net Net-(J7-Pin_1): track 37.8 -> 0.00 mm, vias 1 -> 0
- net SDA: track 171.7 -> 138.8 mm, vias 3 -> 7
- net row4: track 252.7 -> 232.9 mm, vias 10 -> 3
- net +3V3: track 229.7 -> 210.1 mm
- net Net-(D20-Pad2): track 13.2 -> 0.00 mm, vias 1 -> 0
- net col2: track 173.1 -> 163.6 mm
- net col4: track 133.9 -> 128.3 mm
- net row0: track 169.2 -> 164.6 mm, vias 6 -> 0
- net col1: track 194.6 -> 198.5 mm
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Other:
- outline, holes or cut-outs redrawn
- board text added: "DNP:hand"
- board text added: "JLCJLCJLCJLC"
