File: file/pcb/v2/5x6/TPS/TPS.kicad_sch (KiCad schematic)
At the start: 106 parts, among them J1 I2C, J10 AudioJack4, J2 FFC-0.5mm, 12p, J3 FFC-0.5mm, 12p, J4 PH2.0-2pin, J5 FFC-0.5mm, 6p, J6 FFC-0.5mm, 6p, J9 AudioJack4, K1 SW_Push, K10 SW_Push, K11 SW_Push, K12 SW_Push, K13 SW_Push, K14 SW_Push, K15 SW_Push, K16 SW_Push, K17 SW_Push, K18 SW_Push, K19 SW_Push, K2 SW_Push, K20 SW_Push, K21 SW_Push, K22 SW_Push, K23 SW_Push, K24 SW_Push, K25 EC-11, K26 SW_Push, K27 SW_Push, K28 SW_Push, K29 SW_Push, K3 SW_Push, K30 SW_Push, K31 SW_Push, K4 SW_Push, K5 SW_Push, K6 SW_Push, K7 SW_Push, K8 SW_Push, K9 SW_Push, SW1 SW_Push, SW2 MSKT-12D14, SW3 MSKT-12D14, U1 MCU_ProMicro_13p

Commit message: manufacturered with JLCPCB
Parts:
- removed K20: SW_Push, DreaM117er-keebLibrary:SW_Hotswap_KLP12_GLP3.0_MX_Plated_1.00u_Dualside, symbol Switch:SW_Push
- added HM1, HM2, HM3, HM4, HM5, HM6: MountingHole, ncParts:MountingHole_2.2mm_M2_ISO7380_Pad_noSilk, symbol Mechanical:MountingHole
- K1, K11, K12, K13, K14, K15, K16, K17, K18, K19, K2, K21, K22, K23, K24, K27, K28, K29, K3, K30, K4, K6, K7, K8, K9: footprint DreaM117er-keebLibrary:SW_Hotswap_KLP12_GLP3.0_MX_Plated_1.00u_Dualside -> ncSwitches:SW_hotswap_HLP_Plated_1u-reversible
- K10, K26, K31, K5: footprint DreaM117er-keebLibrary:SW_Hotswap_KLP12_GLP3.0_MX_Plated_1.00u_Dualside -> ncSwitches:SW_hotswap_HLP_Plated_1.25u-reversible
Connections:
- net +3V3: now also J5.4 (Pin_4), J6.4 (Pin_4); no longer J5.3 (Pin_3), J6.3 (Pin_3)
- net BAT+: now also J4.1 (Pin_1), J7.1 (Pin_1), J8.2 (Pin_2), SW2.2 (B), SW3.2 (B); no longer SW2.1 (A), SW3.1 (A), U1.26 (?)
- net GND: now also J4.2 (Pin_2), J5.3 (Pin_3), J6.3 (Pin_3), J7.2 (Pin_2), J8.1 (Pin_1); no longer J5.4 (Pin_4), J5.7 (Pin_7), J6.4 (Pin_4), J6.7 (Pin_7)
- net RAW: now also SW2.1 (A), SW3.1 (A)
- net SCL: now also J5.5 (Pin_5), J6.5 (Pin_5); no longer J5.2 (Pin_2), J6.2 (Pin_2)
- net SDA: now also J5.6 (Pin_6), J6.6 (Pin_6); no longer J5.1 (Pin_1), J6.1 (Pin_1)
- net col2: now also D20.2
- removed net BAT-: J4.2 (Pin_2), J7.2 (Pin_2), J8.1 (Pin_1), U1.1 (?)
- no-connect marks 20 -> 24
Other:
- moved on the sheet: J5, J6
